Commit message: original urdf copy from theconstructsim cozmo_simulation package -> https://rds.theconstructsim.com/r/830420c6168e/cozmo_simulation_3__4dca/

File: urdf/vector.urdf.xacro (robot description, xacro)
@@ -1,4 +1,394 @@
-<?xml version="1.0" encoding="UTF-8" ?>
-<robot name="vector" xmlns:xacro="http://ros.org/wiki/xacro">
-    <link name="base_link" />
+<?xml version="1.0" encoding="UTF-8"?>
+<robot name="Vector" xmlns:xacro="http://ros.org/wiki/xacro">
+  <!--XACRO for intertial -->
+  <xacro:macro name="cylinder_inertial" params="radius length mass">
+    <inertial>
+      <mass value="${mass}" />
+      <inertia ixx="${0.0833333 * mass * (3 * radius * radius + length * length)}" ixy="0.0" ixz="0.0"
+        izz="${0.0833333 * mass * (3 * radius * radius + length * length)}" iyz="0.0"
+        iyy="${0.5 * mass * radius * radius}" />
+    </inertial>
+  </xacro:macro>
+  <xacro:macro name="box_inertial" params="mass x y z">
+    <inertial>
+      <mass value="${mass}" />
+      <inertia  ixx="${mass*(y*y+z*z)/12}" ixy = "0" ixz = "0" iyy="${mass*(x*x+z*z)/12}" iyz = "0" izz="${mass*(x*x+z*z)/12}" />
+    </inertial>
+  </xacro:macro>
+    <xacro:macro name="box_inertial_default" params="mass">
+    <inertial>
+      <mass value="${mass}" />
+      <inertia  ixx="0.000001" ixy = "0" ixz = "0" iyy="0.000001" iyz = "0" izz="0.0000001" />
+    </inertial>
+  </xacro:macro>
+  <!-- LINKS ===========================  -->
+  <!--chassis-->
+  <link name="base_link">
+    <xacro:box_inertial mass="0.06" x="0.073" y="0.043" z="0.061" />
+    <visual>
+      <geometry>
+        <mesh filename="package://cozmo_description/meshes/body3.dae"  />
+      </geometry>
+    </visual>
+    <collision>
+      <geometry>
+        <mesh filename="package://cozmo_description/meshes/body3.dae"  />
+      </geometry>
+    </collision>
+  </link>
+  <!--Front left wheel-->
+  <link name="front_left_wheel">
+    <xacro:cylinder_inertial mass="0.005" radius="0.01314" length="0.01167"/>
+    <visual>
+      <geometry>
+        <mesh filename="package://cozmo_description/meshes/flw2.dae"  />
+      </geometry>
+    </visual>
+    <collision>
+      <geometry>
+        <mesh filename="package://cozmo_description/meshes/flw2.dae"  />
+      </geometry>
+    </collision>
+  </link>
+  <!--Front right wheel  -->
+  <link name="front_right_wheel">
+    <xacro:cylinder_inertial mass="0.005" radius="0.01314" length="0.01167"/>
+    <visual>
+      <geometry>
+        <mesh filename="package://cozmo_description/meshes/flw2.dae"/>
+      </geometry>
+    </visual>
+    <collision>
+      <geometry>
+        <mesh filename="package://cozmo_description/meshes/flw2.dae"/>
+      </geometry>
+    </collision>
+  </link>
+  <!--Rear left wheel -->
+  <link name="rear_left_wheel">
+    <xacro:cylinder_inertial mass="0.005" radius="0.008995" length="0.01167"/>
+    <visual>
+      <geometry>
+        <mesh filename="package://cozmo_description/meshes/rlw2.dae" />
+      </geometry>
+    </visual>
+    <collision>
+      <geometry>
+        <mesh filename="package://cozmo_description/meshes/rlw2.dae"/>
+      </geometry>
+    </collision>
+  </link>
+  <!--Rear right wheel -->
+  <link name="rear_right_wheel">
+    <xacro:cylinder_inertial mass="0.005" radius="0.008995" length="0.01167"/>
+    <visual>
+      <geometry>
+        <mesh filename="package://cozmo_description/meshes/rlw2.dae"/>
+      </geometry>
+    </visual>
+    <collision>
+      <geometry>
+        <mesh filename="package://cozmo_description/meshes/rlw2.dae"/>
+      </geometry>
+    </collision>
+  </link>
+  <!-- Head -->
+  <link name="head">
+    <xacro:box_inertial mass="0.01" x="0.036" y="0.038" z="0.041" />
+    <visual>
+      <geometry>
+        <mesh filename="package://cozmo_description/meshes/head_screen.dae" />
+      </geometry>
+    </visual>
+    <collision>
+      <geometry>
+        <mesh filename="package://cozmo_description/meshes/head_screen.dae"/>
+      </geometry>
+    </collision>
+  </link>
+  <!-- lifter -->
+  <link name="full_lift">
+    <inertial>
+      <origin xyz="0.025 0 0"/>
+      <mass value="0.01" />
+      <inertia  ixx="0.000004887" ixy = "0" ixz = "0" iyy="0.000007551" iyz = "0" izz="0.000007551" />
+    </inertial>
+    <!-- <xacro:box_inertial mass="0.01" x="0.081" y="0.058" z="0.050"/> -->
+    <visual>
+      <geometry>
+        <mesh filename="package://cozmo_description/meshes/lift3.dae"/>
+      </geometry>
+    </visual>
+    <collision>
+      <geometry>
+        <mesh filename="package://cozmo_description/meshes/lift3.dae"/>
+      </geometry>
+    </collision>
+  </link>
+  <!-- Belts -->
+  <link name="left_belt">
+    <xacro:box_inertial_default mass="0.0001"/>
+    <visual>
+      <geometry>
+        <mesh filename="package://cozmo_description/meshes/belt.dae" />
+      </geometry>
+    </visual>
+  </link>
+  <link name="right_belt">
+    <xacro:box_inertial_default mass="0.0001"/>
+    <visual>
+      <geometry>
+        <mesh filename="package://cozmo_description/meshes/belt.dae" />
+      </geometry>
+    </visual>
+  </link>
+  <!-- sensors links -->
+  <link name="camera_link">
+    <visual>
+      <geometry>
+        <box size="0.005 0.005 0.005"/>
+      </geometry>
+    </visual>
+  </link>
+  <link name="drop_ir">
+    <visual>
+      <geometry>
+        <box size="0.005 0.005 0.005"/>
+      </geometry>
+    </visual>
+  </link>
+<!--
+  <link name="imu">
+    <visual>
+      <geometry>
+        <box size="0.005 0.005 0.005"/>
+      </geometry>
+    </visual>
+  </link>
+-->
+  <!-- JOINTS ====================================-->
+   <joint name="base_to_lift" type="revolute">
+    <parent link="base_link"/>
+    <child link="full_lift"/>
+    <origin xyz="-0.005 0 0.013"/>
+    <limit lower="-0.8" upper="0" effort="5" velocity="10"/>
+    <axis xyz="0 1 0"/>
+  </joint>
+  <joint name="base_to_head" type="revolute">
+    <parent link="base_link"/>
+    <child link="head"/>
+    <origin xyz="0.015 0 0.02"/>
+    <limit lower="-0.52" upper="0.17" effort="100" velocity="10"/>
+    <dynamics damping="10" friction="1"/>
+    <axis xyz="0 1 0"/>
+  </joint>
+  <joint name="base_to_flw" type="continuous">
+    <parent link="base_link"/>
+    <child link="front_left_wheel"/>
+    <origin xyz="0.03 0.024 -0.012"/>
+    <axis xyz="0 1 0"/>
+  </joint>
+  <joint name="base_to_frw" type="continuous">
+    <parent link="base_link"/>
+    <child link="front_right_wheel"/>
+    <origin xyz="0.03 -0.024 -0.012"/>
+    <axis xyz="0 1 0"/>
+  </joint>
+  <joint name="base_to_rlw" type="continuous">
+    <parent link="base_link"/>
+    <child link="rear_left_wheel"/>
+    <origin xyz="-0.017 0.024 -0.012"/>
+    <axis xyz="0 1 0"/>
+  </joint>
+  <joint name="base_to_rrw" type="continuous">
+    <parent link="base_link"/>
+    <child link="rear_right_wheel"/>
+    <origin xyz="-0.017 -0.024 -0.012"/>
+    <axis xyz="0 1 0"/>
+  </joint>
+   <joint name="head_camera_joint" type="fixed">
+    <parent link="head"/>
+    <child link="camera_link"/>
+    <origin xyz="0.07 0 0.0" rpy="0 0 0"/>
+  </joint>
+  <joint name="drop_ir_joint" type="fixed">
+    <parent link="base_link"/>
+    <child link="drop_ir"/>
+    <origin xyz="0 0 0" rpy="0 1.57 0" />
+  </joint>
+<!--
+  <joint name="imu_joint" type="fixed">
+    <parent link="head"/>
+    <child link="imu"/>
+    <origin xyz="0.0 0 0.0" rpy="0 0 0" />
+  </joint>
+-->
+  <joint name="wheel_left_belt" type="fixed">
+    <parent link="base_link"/>
+    <child link="left_belt"/>
+    <origin xyz="0.01 0.024 -0.012"/>
+  </joint>
+  <joint name="wheel_right_belt" type="fixed">
+    <parent link="base_link"/>
+    <child link="right_belt"/>
+    <origin xyz="0.01 -0.024 -0.012"/>
+  </joint>
+  <!-- Transmissions for joints -->
+    <transmission name="base_to_head_trans">
+      <type>transmission_interface/SimpleTransmission</type>
+      <joint name="base_to_head">
+        <hardwareInterface>hardware_interface/EffortJointInterface</hardwareInterface>
+      </joint>
+      <actuator name="base_to_headMotor">
+        <hardwareInterface>hardware_interface/EffortJointInterface</hardwareInterface>
+        <mechanicalReduction>1</mechanicalReduction>
+      </actuator>
+  </transmission>
+  <transmission name="base_to_lift_trans">
+      <type>transmission_interface/SimpleTransmission</type>
+      <joint name="base_to_lift">
+        <hardwareInterface>hardware_interface/EffortJointInterface</hardwareInterface>
+      </joint>
+      <actuator name="base_to_liftMotor">
+        <hardwareInterface>hardware_interface/EffortJointInterface</hardwareInterface>
+        <mechanicalReduction>1</mechanicalReduction>
+      </actuator>
+  </transmission>
+    <!--                GAZEBO RELATED PART                             -->
+  <!-- ROS Control plugin for Gazebo -->
+  <gazebo>
+    <plugin name="gazebo_ros_control" filename="libgazebo_ros_control.so">
+      <robotNamespace>/cozmo</robotNamespace>
+    </plugin>
+  </gazebo>
+  <gazebo reference="camera_link">
+    <sensor type="camera" name="cozmo_camera">
+      <update_rate>10.0</update_rate>
+      <camera name="headcamera">
+        <horizontal_fov>1.3962634</horizontal_fov>
+        <image>
+          <width>400</width>
+          <height>400</height>
+          <format>R8G8B8</format>
+        </image>
+        <clip>
+          <near>0.01</near>
+          <far>100</far>
+        </clip>
+        <noise>
+          <type>gaussian</type>
+          <mean>0.0</mean>
+          <stddev>0.007</stddev>
+        </noise>
+      </camera>
+      <plugin name="camera_controller" filename="libgazebo_ros_camera.so">
+        <alwaysOn>true</alwaysOn>
+        <updateRate>10.0</updateRate>
+        <cameraName>cozmo_camera</cameraName>
+        <imageTopicName>image</imageTopicName>
+        <cameraInfoTopicName>camera_info</cameraInfoTopicName>
+        <frameName>camera_link</frameName>
+        <hackBaseline>0.07</hackBaseline>
+        <distortionK1>0.0</distortionK1>
+        <distortionK2>0.0</distortionK2>
+        <distortionK3>0.0</distortionK3>
+        <distortionT1>0.0</distortionT1>
+        <distortionT2>0.0</distortionT2>
+      </plugin>
+    </sensor>
+  </gazebo>
+<gazebo reference="drop_ir">
+ <sensor type="ray" name="TeraRanger">
+    <pose>0 0 0 0 0 0</pose>
+    <visualize>true</visualize>
+    <update_rate>50</update_rate>
+    <ray>
+       <scan>
+          <horizontal>
+             <samples>10</samples>
+             <resolution>1</resolution>
+             <min_angle>-0.14835</min_angle>
+             <max_angle>0.14835</max_angle>
+          </horizontal>
+          <vertical>
+             <samples>10</samples>
+             <resolution>1</resolution>
+             <min_angle>-0.14835</min_angle>
+             <max_angle>0.14835</max_angle>
+          </vertical>
+       </scan>
+       <range>
+          <min>0.01</min>
+          <max>2</max>
+          <resolution>0.02</resolution>
+       </range>
+    </ray>
+    <plugin filename="libgazebo_ros_range.so" name="gazebo_ros_range">
+       <gaussianNoise>0.005</gaussianNoise>
+       <alwaysOn>true</alwaysOn>
+       <updateRate>50</updateRate>
+       <topicName>drop_sensor</topicName>
+       <frameName>drop_ir</frameName>
+       <radiation>INFRARED</radiation>
+       <fov>0.2967</fov>
+    </plugin>
+ </sensor>
+ </gazebo>
+ <!--IMU gazebo-->
+ <gazebo reference="imu">
+    <gravity>true</gravity>
+    <sensor name="imu_sensor" type="imu">
+      <always_on>true</always_on>
+      <update_rate>100</update_rate>
+      <visualize>true</visualize>
+      <topic>__default_topic__</topic>
+      <plugin filename="libgazebo_ros_imu_sensor.so" name="imu_plugin">
+        <topicName>imu</topicName>
+        <bodyName>imu</bodyName>
+        <updateRateHZ>10.0</updateRateHZ>
+        <gaussianNoise>${0.0017*0.0017}</gaussianNoise>
+        <xyzOffset>0 0 0</xyzOffset>
+        <rpyOffset>0 0 0</rpyOffset>
+        <frameName>imu</frameName>
+      </plugin>
+      <pose>0 0 0 0 0 0</pose>
+    </sensor>
+  </gazebo>
+<!--
+  <gazebo reference="rear_right_wheel">
+    <mu1>100000</mu1>
+    <mu2>100000</mu2>
+  </gazebo>
+  <gazebo reference="rear_left_wheel">
+    <mu1>100000</mu1>
+    <mu2>100000</mu2>
+  </gazebo>
+<gazebo reference="front_right_wheel">
+    <mu1>100000</mu1>
+    <mu2>100000</mu2>
+  </gazebo>
+  <gazebo reference="front_left_wheel">
+    <mu1>100000</mu1>
+    <mu2>100000</mu2>
+  </gazebo>
+-->
+  <gazebo>
+  <plugin name="skid_steer_drive_controller" filename="libgazebo_ros_skid_steer_drive.so">
+    <updateRate>25.0</updateRate>
+    <robotNamespace>/</robotNamespace>
+    <leftFrontJoint>base_to_flw</leftFrontJoint>
+    <rightFrontJoint>base_to_frw</rightFrontJoint>
+    <leftRearJoint>base_to_rlw</leftRearJoint>
+    <rightRearJoint>base_to_rrw</rightRearJoint>
+    <wheelSeparation>0.048</wheelSeparation>
+    <wheelDiameter>0.04</wheelDiameter>
+    <robotBaseFrame>base_link</robotBaseFrame>
+    <torque>20</torque>
+    <topicName>cmd_vel</topicName>
+    <commandTopic>cmd_vel</commandTopic>
+    <odometryTopic>odom</odometryTopic>
+    <odometryFrame>odom</odometryFrame>
+    <broadcastTF>1</broadcastTF>
+  </plugin>
+  </gazebo>
 </robot>
